File: sch/led-controller.sch (KiCad schematic (older format))
At the start: 8 parts, among them P1 CONN_2, P2 CONN_4, P3 CONN_2, U1 ATTINY4

Commit message: fixed some problems with the pcb and schematic.
Parts:
- removed P1, P3: CONN_2, symbol CONN_2
- added K1: GND, symbol CONN_3
- added K2: VCC, symbol CONN_3
- D1: value RGB_LED -> LED
- P2: value CONN_4 -> IO
- U1: value ATTINY4 -> MCU
Connections:
- net labels added: VCC
- wire segments 23 -> 24
Changed lines of the file:
@@
-EESchema Schematic File Version 2  date Tue 28 Feb 2012 07:49:53 PM PST
+EESchema Schematic File Version 2  date Sun 01 Apr 2012 11:15:49 AM PDT
 LIBS:power
 LIBS:device
@@
 Sheet 1 1
 Title ""
-Date "29 feb 2012"
+Date "1 apr 2012"
 Rev ""
 Comp ""
@@
 Comment4 ""
 $EndDescr
+$Comp
+L CONN_3 K1
+U 1 1 4F789AEC
+P 2600 3850
+F 0 "K1" V 2550 3850 50  0000 C CNN
+F 1 "GND" V 2650 3850 40  0000 C CNN
+	1    2600 3850
+	-1   0    0    1
+$EndComp
+$Comp
+L CONN_3 K2
+U 1 1 4F789ADE
+P 7250 3850
+F 0 "K2" V 7200 3850 50  0000 C CNN
+F 1 "VCC" V 7300 3850 40  0000 C CNN
+	1    7250 3850
+	1    0    0    -1
+$EndComp
+Connection ~ 3400 3850
+Wire Wire Line
+	3400 4300 3400 3850
+Connection ~ 6900 3850
+Wire Wire Line
+	5750 3850 6900 3850
+Wire Wire Line
+	2950 3950 2950 3750
+Wire Wire Line
+	5450 2950 5050 2950
+Wire Wire Line
+	5050 2950 5050 2700
+Wire Wire Line
+	4500 2800 4850 2800
+Wire Wire Line
+	4850 2800 4850 2700
+Wire Wire Line
+	4250 3950 4000 3950
+Wire Wire Line
+	6000 3750 5750 3750
+Wire Wire Line
+	4250 5350 4100 5350
+Wire Wire Line
+	5750 5350 5950 5350
+Wire Wire Line
+	4250 4450 4100 4450
+Wire Wire Line
+	4250 3250 4100 3250
+Wire Wire Line
+	5750 4450 5900 4450
+Wire Wire Line
+	5750 5450 5950 5450
+Wire Wire Line
+	4250 5450 4100 5450
+Wire Wire Line
+	5750 3950 6000 3950
+Wire Wire Line
+	4250 3750 4000 3750
+Wire Wire Line
+	4950 2700 4950 2950
+Wire Wire Line
+	4950 2950 4500 2950
+Wire Wire Line
+	5150 2700 5150 2800
+Wire Wire Line
+	5150 2800 5450 2800
+Wire Wire Line
+	6900 3750 6900 3950
+Wire Wire Line
+	4250 3850 2950 3850
 Connection ~ 2950 3850
-Wire Wire Line
-	4250 3850 2950 3850
-Wire Wire Line
-	6900 3950 6900 3750
-Wire Wire Line
-	5450 2800 5150 2800
-Wire Wire Line
-	5150 2800 5150 2700
-Wire Wire Line
-	4500 2950 4950 2950
-Wire Wire Line
-	4950 2950 4950 2700
-Wire Wire Line
-	4250 3750 4000 3750
-Wire Wire Line
-	5750 3950 6000 3950
-Wire Wire Line
-	4250 5450 4100 5450
-Wire Wire Line
-	5750 5450 5950 5450
-Wire Wire Line
-	5750 4450 5900 4450
-Wire Wire Line
-	4250 3250 4100 3250
-Wire Wire Line
-	4250 4450 4100 4450
-Wire Wire Line
-	5750 5350 5950 5350
-Wire Wire Line
-	4250 5350 4100 5350
-Wire Wire Line
-	6000 3750 5750 3750
-Wire Wire Line
-	4250 3950 4000 3950
-Wire Wire Line
-	4850 2700 4850 2800
-Wire Wire Line
-	4850 2800 4500 2800
-Wire Wire Line
-	5050 2700 5050 2950
-Wire Wire Line
-	5050 2950 5450 2950
-Wire Wire Line
-	2950 3750 2950 3950
-Wire Wire Line
-	5750 3850 6900 3850
-Connection ~ 6900 3850
+Text Label 3150 3850 0    60   ~ 0
+GND
+Text Label 6600 3850 0    60   ~ 0
+VCC
+$Comp
+L GND #PWR1
+U 1 1 4F78907D
+P 3400 4300
+F 0 "#PWR1" H 3400 4300 30  0001 C CNN
+F 1 "GND" H 3400 4230 30  0001 C CNN
+	1    3400 4300
+	1    0    0    -1
+$EndComp
 Text Label 5450 2950 2    60   ~ 0
 PB2
@@
 BLUE
 $Comp
-L GND #PWR01
+L GND #PWR2
 U 1 1 4F4D9E75
 P 4100 5450
-F 0 "#PWR01" H 4100 5450 30  0001 C CNN
+F 0 "#PWR2" H 4100 5450 30  0001 C CNN
 F 1 "GND" H 4100 5380 30  0001 C CNN
 	1    4100 5450
@@
 P 5000 2350
 F 0 "P2" V 4950 2350 50  0000 C CNN
-F 1 "CONN_4" V 5050 2350 50  0000 C CNN
+F 1 "IO" V 5050 2350 50  0000 C CNN
 	1    5000 2350
 	0    -1   -1   0
-$EndComp
-$Comp
-L CONN_2 P1
-U 1 1 4F4D9D49
-P 2600 3850
-F 0 "P1" V 2550 3850 40  0000 C CNN
-F 1 "CONN_2" V 2650 3850 40  0000 C CNN
-	1    2600 3850
-	-1   0    0    1
-$EndComp
-$Comp
-L CONN_2 P3
-U 1 1 4F4D9D46
-P 7250 3850
-F 0 "P3" V 7200 3850 40  0000 C CNN
-F 1 "CONN_2" V 7300 3850 40  0000 C CNN
-	1    7250 3850
-	1    0    0    -1
 $EndComp
 $Comp
@@
 P 5000 5400
 F 0 "D1" H 5000 5300 50  0000 C CNN
-F 1 "RGB_LED" H 5000 5500 50  0000 C CNN
+F 1 "LED" H 5000 5500 50  0000 C CNN
 F 2 "MODULE" H 5000 5400 50  0001 C CNN
 F 3 "DOCUMENTATION" H 5000 5400 50  0001 C CNN
@@
 P 5000 3850
 F 0 "U1" H 5000 3750 50  0000 C CNN
-F 1 "ATTINY4" H 5000 3950 50  0000 C CNN
+F 1 "MCU" H 5000 3950 50  0000 C CNN
 F 2 "MODULE" H 5000 3850 50  0001 C CNN
 F 3 "DOCUMENTATION" H 5000 3850 50  0001 C CNN
